File: Hardware/OpenBook-board.brd (EAGLE design)
At the start: 170.2 x 111.2 mm, 103 parts, among them IC1 BD5229G-TR, IC4 XC6220A331MR-G, J1 FH34SRJ-24S-0.5SH_99_, J2 SAMACSYS_PARTS_USB4110-GF-A, J3 QWIIC_RIGHT_ANGLE, J4 112A-TAAR-R03_ATTEND3DMODEL, Q1 20V/4.2A/52mΩ/1.4W, Q2 20V/4.2A/52mΩ/1.4W, Q3 SI1308EDL-T1-GE3, U1 W25Q512JVEIQ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

Commit message: solved ESP32 issue
Routing:
- net SS_SD: track 63.9 -> 66.0 mm
- net GND: track 734.0 -> 735.0 mm
- net SCK: track 231.4 -> 230.7 mm
Other:
- outline, holes or cut-outs redrawn
